Commit message: 4 wheels box

File: description/robot_core.xacro (robot description, xacro)
@@ -24,8 +24,72 @@
         <origin xyz="0.1 0 0.045"/>
             <geometry>
-                <box size="0.2 0.15 0.09"/>
+                <box size="0.2 0.11 0.1"/>
             </geometry>
             <material name="white"/>
        </visual>
     </link>
+    <!--Left-Front Wheel-->
+    <joint name="left_front_wheel_joint" type="continuous">
+        <parent link="base_link"/>
+        <child link="left_front_wheel"/>
+        <origin xyz="0.047 0.065 0" rpy="-${pi/2} 0 0"/>
+        <axis xyz="0 0 1"/>
+    </joint>
+    <link name="left_front_wheel">
+        <visual>
+            <origin xyz="0 0 0" rpy="0 0 0"/>
+            <geometry>
+                <cylinder length="0.02" radius="0.0235"/>
+            </geometry>
+            <material name="black"/>
+        </visual>
+    </link>
+    <!--Right-Front Wheel-->
+    <joint name="right_front_wheel_joint" type="continuous">
+        <parent link="base_link"/>
+        <child link="right_front_wheel"/>
+        <origin xyz="0.047 -0.065 0" rpy="${pi/2} 0 0"/>
+        <axis xyz="0 0 -1"/>
+    </joint>
+    <link name="right_front_wheel">
+        <visual>
+            <origin xyz="0 0 0" rpy="0 0 0"/>
+            <geometry>
+                <cylinder length="0.02" radius="0.0235"/>
+            </geometry>
+            <material name="black"/>
+        </visual>
+    </link>
+    <!--Left-Back Wheel-->
+    <joint name="left_back_wheel_joint" type="continuous">
+        <parent link="base_link"/>
+        <child link="left_back_wheel"/>
+        <origin xyz="-0.047 0.065 0" rpy="-${pi/2} 0 0"/>
+        <axis xyz="0 0 1"/>
+    </joint>
+    <link name="left_back_wheel">
+        <visual>
+            <origin xyz="0 0 0" rpy="0 0 0"/>
+            <geometry>
+                <cylinder length="0.02" radius="0.0235"/>
+            </geometry>
+            <material name="black"/>
+        </visual>
+    </link>
+    <!--Right-back Wheel-->
+    <joint name="right_back_wheel_joint" type="continuous">
+        <parent link="base_link"/>
+        <child link="right_back_wheel"/>
+        <origin xyz="-0.047 -0.065 0" rpy="${pi/2} 0 0"/>
+        <axis xyz="0 0 -1"/>
+    </joint>
+    <link name="right_back_wheel">
+        <visual>
+            <origin xyz="0 0 0" rpy="0 0 0"/>
+            <geometry>
+                <cylinder length="0.02" radius="0.0235"/>
+            </geometry>
+            <material name="black"/>
+        </visual>
+    </link>
 </robot>

Commit message: adding masses

File: description/robot_core.xacro (robot description, xacro)
@@ -1,4 +1,5 @@
 <?xml version="1.0"?>
 <robot xmlns:xacro="http://www.ros.org/wiki/xacro" >
+    <xacro:include filename="inertial_macros.xacro" />
     <material name="white">
         <color rgba="1 1 1 1" />
@@ -28,4 +29,13 @@
             <material name="white"/>
        </visual>
+        <collision>
+        <origin xyz="0.1 0 0.045"/>
+            <geometry>
+                <box size="0.2 0.11 0.1"/>
+            </geometry>
+        </collision>
+        <xacro:inertial_box mass="1.5" x="0.2" y="0.11" z="0.1">
+            <origin xyz="0.1 0 0.045" rpy="0 0 0"/>
+        </xacro:inertial_box>
     </link>
     <!--Left-Front Wheel-->
@@ -44,4 +54,13 @@
             <material name="black"/>
         </visual>
+        <collision>
+            <origin xyz="0 0 0" rpy="0 0 0"/>
+            <geometry>
+                <cylinder length="0.02" radius="0.0235"/>
+            </geometry>
+        </collision>
+        <xacro:inertial_cylinder mass="0.05" length="0.02" radius="0.0235">
+            <origin xyz="0 0 0" rpy="0 0 0"/>
+        </xacro:inertial_cylinder>
     </link>
     <!--Right-Front Wheel-->
@@ -60,4 +79,13 @@
             <material name="black"/>
         </visual>
+        <collision>
+            <origin xyz="0 0 0" rpy="0 0 0"/>
+            <geometry>
+                <cylinder length="0.02" radius="0.0235"/>
+            </geometry>
+        </collision>
+        <xacro:inertial_cylinder mass="0.05" length="0.02" radius="0.0235">
+            <origin xyz="0 0 0" rpy="0 0 0"/>
+        </xacro:inertial_cylinder>
     </link>
     <!--Left-Back Wheel-->
@@ -76,4 +104,13 @@
             <material name="black"/>
         </visual>
+        <collision>
+            <origin xyz="0 0 0" rpy="0 0 0"/>
+            <geometry>
+                <cylinder length="0.02" radius="0.0235"/>
+            </geometry>
+        </collision>
+        <xacro:inertial_cylinder mass="0.05" length="0.02" radius="0.0235">
+            <origin xyz="0 0 0" rpy="0 0 0"/>
+        </xacro:inertial_cylinder>
     </link>
     <!--Right-back Wheel-->
@@ -92,4 +129,13 @@
             <material name="black"/>
         </visual>
+        <collision>
+            <origin xyz="0 0 0" rpy="0 0 0"/>
+            <geometry>
+                <cylinder length="0.02" radius="0.0235"/>
+            </geometry>
+        </collision>
+        <xacro:inertial_cylinder mass="0.05" length="0.02" radius="0.0235">
+            <origin xyz="0 0 0" rpy="0 0 0"/>
+        </xacro:inertial_cylinder>
     </link>
 </robot>
